File: hardware/pcb/top/top.kicad_pcb (KiCad board)
At the start: 2 copper layers, 65 x 120 mm, 33 parts, among them J1 OLED_128x32, J2 Conn_01x15, SW1 SLW-864574-5A-RA-N-D, SW2 RotaryEncoder_Switch

Commit message: fixed grounding vias cutting column pads and updated name and rev number
Routing:
- net GND: vias 145 -> 143
Other:
- board text added: "ApexPad"
- board text added: "Rev 1.1"
- board text removed: "Proiect Licenta - Macropad -"
- board text removed: "Realizat de Pal Antonio"
- board text removed: "Rev 1.0"
Changed lines of the file:
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@@
 		(layer "Edge.Cuts")
 	)
-	(gr_text "Proiect Licenta\n- Macropad -"
-		(at 166.78493 30.93882 0)
+	(gr_text "ApexPad"
+		(at 167.53493 31.43882 0)
 		(layer "F.SilkS")
 		(effects
 			(font
-				(size 1 1)
-				(thickness 0.2)
+				(size 2 2)
+				(thickness 0.4)
 				(bold yes)
 			)
 		)
 	)
-	(gr_text "Rev 1.0"
-		(at 176.28493 36.93882 0)
+	(gr_text "Rev 1.1"
+		(at 167.78493 35.18882 0)
 		(layer "F.SilkS")
 		(effects
 			(font
-				(size 1 1)
-				(thickness 0.2)
+				(size 2 2)
+				(thickness 0.4)
 				(bold yes)
 			)
 		)
 	)
-	(gr_text "Realizat de Pal Antonio"
-		(at 170.28493 34.43882 0)
-		(layer "F.SilkS")
-		(effects
-			(font
-				(size 1 1)
-				(thickness 0.2)
-				(bold yes)
-			)
-		)
-	)
 	(segment
 		(start 163.28493 110.12493)
@@
 	)
 	(via
-		(at 126.53493 109.94618)
-		(size 0.6)
-		(drill 0.3)
-		(layers "F.Cu" "B.Cu")
-		(free yes)
-		(net 22)
-	)
-	(via
 		(at 131.53493 79.18882)
 		(size 0.6)
@@
 		(size 0.6)
 		(drill 0.3)
-		(layers "F.Cu" "B.Cu")
-		(free yes)
-		(net 22)
-	)
-	(via
-		(at 136.53493 89.94618)
-		(size 0.6)
-		(drill 0.3)
